Commit message: teste da classe ManipulatorIK com rosparams para cinemática inversa funcionando para ser inclusa e usada em outros .cpp

File: manipulator_description/urdf/urdf_remade.urdf.xacro (robot description, xacro)
@@ -340,11 +340,11 @@
       velocity="2" />
   </joint>
-  <link name="air" />
+  <link name="ee_center" />
    <joint
-    name="joint_gripper_air"
+    name="joint_gripper_ee_center"
     type="fixed">
     <origin xyz="-0.06 0 0.03" rpy="0 0 0" />
     <parent link="gripper" />
-    <child link="air" />
+    <child link="ee_center" />
   </joint>
 </robot>

Commit message: IK está ouvindo tópico transformed da jevois, não estamos encontrando soluções no planning; provalvelmente transform está errado? apenas mudando valores de eixos

File: manipulator_description/urdf/urdf_remade.urdf.xacro (robot description, xacro)
@@ -109,4 +109,24 @@
   </joint>
   <link
+    name="camera">
+    <visual>
+      <geometry>
+        <box size= "0.012 0.012 0.012" />
+      </geometry>
+      <material
+        name="">
+        <color
+          rgba="1.0 0.098039 0.098039 1" />
+      </material>
+    </visual>
+  </link>
+  <joint name="fixed_camera" type="fixed">
+      <origin
+      xyz="0.03 -0.03 0.071"
+      rpy="-1.57 0 0" />
+      <parent link="base_link" />
+      <child link="camera" />
+    </joint>
+  <link
     name="link_1">
     <inertial>
